Commit message: Refactor URDF Xacro for Hexapod: Remove unused properties and standardize RPY values
- Removed mesh orientation correction properties: mesh_up_correction_rpy and mesh_up_correction_with_yaw_rpy.
- Standardized RPY values for base_link, coxa, femur, and tibia links to use fixed values instead of properties.

File: hexapod_ws/src/hexapod_description/urdf/hexapod.urdf.xacro (robot description, xacro)
@@ -5,6 +5,4 @@
   <xacro:property name="tibia_length" value="0.15"/>
   <xacro:property name="femur_z_offset" value="0.0106"/>
-  <xacro:property name="mesh_up_correction_rpy" value="-1.5708 0 0"/>
-  <xacro:property name="mesh_up_correction_with_yaw_rpy" value="-1.5708 0 1.5708"/>
   <!-- ================= MATERIALS ================= -->
   <material name="black"><color rgba="0.1 0.1 0.1 1"/></material>
@@ -18,5 +16,4 @@
   <link name="base_link">
     <visual>
-      <origin xyz="0 0 0" rpy="${mesh_up_correction_rpy}"/>
       <geometry>
         <mesh filename="package://hexapod_description/meshes/body.dae" scale="0.01 0.01 0.01"/>
@@ -25,5 +22,4 @@
     </visual>
     <collision>
-      <origin xyz="0 0 0" rpy="${mesh_up_correction_rpy}"/>
       <geometry>
         <mesh filename="package://hexapod_description/meshes/body.dae" scale="0.01 0.01 0.01"/>
@@ -41,5 +37,5 @@
   <link name="${name}_coxa">
     <visual>
-      <origin xyz="0 0 0" rpy="${mesh_up_correction_with_yaw_rpy}"/>
+      <origin xyz="0 0 0" rpy="0 0 1.5708"/>
       <geometry>
         <mesh filename="package://hexapod_description/meshes/coxa.dae" scale="0.01 0.01 0.01"/>
@@ -48,5 +44,5 @@
     </visual>
     <collision>
-      <origin xyz="0 0 0" rpy="${mesh_up_correction_with_yaw_rpy}"/>
+      <origin xyz="0 0 0" rpy="0 0 1.5708"/>
       <geometry>
         <mesh filename="package://hexapod_description/meshes/coxa.dae" scale="0.01 0.01 0.01"/>
@@ -62,5 +58,5 @@
   <link name="${name}_femur">
     <visual>
-      <origin xyz="0 0 0" rpy="${mesh_up_correction_with_yaw_rpy}"/>
+      <origin xyz="0 0 0" rpy="0 0 1.5708"/>
       <geometry>
         <mesh filename="package://hexapod_description/meshes/femur.dae" scale="0.01 0.01 0.01"/>
@@ -69,5 +65,5 @@
     </visual>
     <collision>
-      <origin xyz="0 0 0" rpy="${mesh_up_correction_with_yaw_rpy}"/>
+      <origin xyz="0 0 0" rpy="0 0 1.5708"/>
       <geometry>
         <mesh filename="package://hexapod_description/meshes/femur.dae" scale="0.01 0.01 0.01"/>
@@ -83,5 +79,5 @@
   <link name="${name}_tibia">
     <visual>
-      <origin xyz="0 0 0" rpy="${mesh_up_correction_with_yaw_rpy}"/>
+      <origin xyz="0 0 0" rpy="0 0 1.5708"/>
       <geometry>
         <mesh filename="package://hexapod_description/meshes/tibia.dae" scale="0.01 0.01 0.01"/>
@@ -90,5 +86,5 @@
     </visual>
     <collision>
-      <origin xyz="0 0 0" rpy="${mesh_up_correction_with_yaw_rpy}"/>
+      <origin xyz="0 0 0" rpy="0 0 1.5708"/>
       <geometry>
         <mesh filename="package://hexapod_description/meshes/tibia.dae" scale="0.01 0.01 0.01"/>

Commit message: Update mesh scaling in URDF: change scale from 0.01 to 1 for body, coxa, femur, and tibia

File: hexapod_ws/src/hexapod_description/urdf/hexapod.urdf.xacro (robot description, xacro)
@@ -17,5 +17,5 @@
     <visual>
       <geometry>
-        <mesh filename="package://hexapod_description/meshes/body.dae" scale="0.01 0.01 0.01"/>
+        <mesh filename="package://hexapod_description/meshes/body.dae" scale="1 1 1"/>
       </geometry>
       <material name="black"/>
@@ -23,5 +23,5 @@
     <collision>
       <geometry>
-        <mesh filename="package://hexapod_description/meshes/body.dae" scale="0.01 0.01 0.01"/>
+        <mesh filename="package://hexapod_description/meshes/body.dae" scale="1 1 1"/>
       </geometry>
     </collision>
@@ -39,5 +39,5 @@
       <origin xyz="0 0 0" rpy="0 0 1.5708"/>
       <geometry>
-        <mesh filename="package://hexapod_description/meshes/coxa.dae" scale="0.01 0.01 0.01"/>
+        <mesh filename="package://hexapod_description/meshes/coxa.dae" scale="1 1 1"/>
       </geometry>
       <material name="${colour}"/>
@@ -46,5 +46,5 @@
       <origin xyz="0 0 0" rpy="0 0 1.5708"/>
       <geometry>
-        <mesh filename="package://hexapod_description/meshes/coxa.dae" scale="0.01 0.01 0.01"/>
+        <mesh filename="package://hexapod_description/meshes/coxa.dae" scale="1 1 1"/>
       </geometry>
     </collision>
@@ -60,5 +60,5 @@
       <origin xyz="0 0 0" rpy="0 0 1.5708"/>
       <geometry>
-        <mesh filename="package://hexapod_description/meshes/femur.dae" scale="0.01 0.01 0.01"/>
+        <mesh filename="package://hexapod_description/meshes/femur.dae" scale="1 1 1"/>
       </geometry>
       <material name="${colour}"/>
@@ -67,5 +67,5 @@
       <origin xyz="0 0 0" rpy="0 0 1.5708"/>
       <geometry>
-        <mesh filename="package://hexapod_description/meshes/femur.dae" scale="0.01 0.01 0.01"/>
+        <mesh filename="package://hexapod_description/meshes/femur.dae" scale="1 1 1"/>
       </geometry>
     </collision>
@@ -81,5 +81,5 @@
       <origin xyz="0 0 0" rpy="0 0 1.5708"/>
       <geometry>
-        <mesh filename="package://hexapod_description/meshes/tibia.dae" scale="0.01 0.01 0.01"/>
+        <mesh filename="package://hexapod_description/meshes/tibia.dae" scale="1 1 1"/>
       </geometry>
       <material name="${colour}"/>
@@ -88,5 +88,5 @@
       <origin xyz="0 0 0" rpy="0 0 1.5708"/>
       <geometry>
-        <mesh filename="package://hexapod_description/meshes/tibia.dae" scale="0.01 0.01 0.01"/>
+        <mesh filename="package://hexapod_description/meshes/tibia.dae" scale="1 1 1"/>
       </geometry>
     </collision>
