Commit message: Replace Servo2040 backend with ST3215 ros2_control and I2C sensor drivers
The Pi 5 now drives Waveshare ST3215 bus servos directly, and reads the
BMI088 IMU and the two INA226 power monitors over I2C.

- Add ST3215System, a ros2_control plugin that sync-writes goal positions
  and sync-reads position, speed and load (published as joint effort)
- Add bmi088_node (sensor_msgs/Imu on imu/data_raw, fused to imu/data by
  imu_filter_madgwick) and ina226_node (sensor_msgs/BatteryState on
  power/left and power/right)
- Share one ros2_control xacro between gazebo, mock and st3215 hardware;
  servo IDs are leg * 10 + joint
- Add hexapod_robot.launch.py; hexapod_fake.launch.py now runs it on
  ros2_control mock hardware
- Remap the Gazebo IMU to /imu/data to match the real robot
- Remove the Servo2040 packet code, the fake hardware node, and the
  PowerStatus, LegContact and ControllerInput messages

Co-Authored-By: Claude Opus 5.5 <noreply@anthropic.com>

File: hexapod_ws/src/hexapod_description/urdf/hexapod.urdf.xacro (robot description, xacro)
@@ -1,4 +1,7 @@
 <robot xmlns:xacro="http://ros.org/wiki/xacro" name="hexapod">
   <xacro:arg name="controllers_file" default=""/>
+  <!-- ros2_control hardware: gazebo, mock or st3215 (see hexapod.ros2_control.xacro) -->
+  <xacro:arg name="hardware" default="mock"/>
+  <xacro:arg name="serial_port" default="/dev/ttyAMA0"/>
   <!-- ================= CONSTANTS ================= -->
   <xacro:property name="coxa_length" value="0.0375"/>
@@ -169,39 +172,20 @@
   <!-- Rear right -->
   <xacro:leg name="leg6" x_offset="-0.06733" y_offset="0.0846" yaw="2.61799" colour="magenta"/>
+  <!-- ================= IMU ================= -->
+  <link name="imu_link"/>
+  <joint name="imu_joint" type="fixed">
+    <parent link="base_link"/>
+    <child link="imu_link"/>
+    <origin xyz="0.0 0.0 0.03" rpy="0 0 0"/>
+  </joint>
   <!-- ================= ROS2 CONTROL ================= -->
-  <xacro:macro name="ros2_control_joint" params="joint_name">
-    <joint name="${joint_name}">
-      <command_interface name="position"/>
-      <state_interface name="position"/>
-      <state_interface name="velocity"/>
-    </joint>
-  </xacro:macro>
-  <ros2_control name="HexapodHardware" type="system">
-    <hardware>
-      <plugin>gz_ros2_control/GazeboSimSystem</plugin>
-    </hardware>
-    <xacro:ros2_control_joint joint_name="leg1_coxa_joint"/>
-    <xacro:ros2_control_joint joint_name="leg1_femur_joint"/>
-    <xacro:ros2_control_joint joint_name="leg1_tibia_joint"/>
-    <xacro:ros2_control_joint joint_name="leg2_coxa_joint"/>
-    <xacro:ros2_control_joint joint_name="leg2_femur_joint"/>
-    <xacro:ros2_control_joint joint_name="leg2_tibia_joint"/>
-    <xacro:ros2_control_joint joint_name="leg3_coxa_joint"/>
-    <xacro:ros2_control_joint joint_name="leg3_femur_joint"/>
-    <xacro:ros2_control_joint joint_name="leg3_tibia_joint"/>
-    <xacro:ros2_control_joint joint_name="leg4_coxa_joint"/>
-    <xacro:ros2_control_joint joint_name="leg4_femur_joint"/>
-    <xacro:ros2_control_joint joint_name="leg4_tibia_joint"/>
-    <xacro:ros2_control_joint joint_name="leg5_coxa_joint"/>
-    <xacro:ros2_control_joint joint_name="leg5_femur_joint"/>
-    <xacro:ros2_control_joint joint_name="leg5_tibia_joint"/>
-    <xacro:ros2_control_joint joint_name="leg6_coxa_joint"/>
-    <xacro:ros2_control_joint joint_name="leg6_femur_joint"/>
-    <xacro:ros2_control_joint joint_name="leg6_tibia_joint"/>
-  </ros2_control>
-  <gazebo>
-    <plugin name="gz_ros2_control::GazeboSimROS2ControlPlugin" filename="libgz_ros2_control-system.so">
-      <parameters>$(arg controllers_file)</parameters>
-    </plugin>
-  </gazebo>
+  <xacro:include filename="$(find hexapod_description)/urdf/hexapod.ros2_control.xacro"/>
+  <xacro:hexapod_ros2_control hardware="$(arg hardware)" serial_port="$(arg serial_port)"/>
+  <xacro:if value="${'$(arg hardware)' == 'gazebo'}">
+    <gazebo>
+      <plugin name="gz_ros2_control::GazeboSimROS2ControlPlugin" filename="libgz_ros2_control-system.so">
+        <parameters>$(arg controllers_file)</parameters>
+      </plugin>
+    </gazebo>
+  </xacro:if>
 </robot>

File: hexapod_ws/src/hexapod_description/urdf/hexapod_primitives.urdf.xacro (robot description, xacro)
@@ -352,34 +352,6 @@
 </gazebo>
   <!-- ================= ROS2 CONTROL ================= -->
-  <xacro:macro name="ros2_control_joint" params="joint_name">
-    <joint name="${joint_name}">
-      <command_interface name="position"/>
-      <state_interface name="position"/>
-      <state_interface name="velocity"/>
-    </joint>
-  </xacro:macro>
-  <ros2_control name="HexapodHardware" type="system">
-    <hardware>
-      <plugin>gz_ros2_control/GazeboSimSystem</plugin>
-    </hardware>
-    <xacro:ros2_control_joint joint_name="leg1_coxa_joint"/>
-    <xacro:ros2_control_joint joint_name="leg1_femur_joint"/>
-    <xacro:ros2_control_joint joint_name="leg1_tibia_joint"/>
-    <xacro:ros2_control_joint joint_name="leg2_coxa_joint"/>
-    <xacro:ros2_control_joint joint_name="leg2_femur_joint"/>
-    <xacro:ros2_control_joint joint_name="leg2_tibia_joint"/>
-    <xacro:ros2_control_joint joint_name="leg3_coxa_joint"/>
-    <xacro:ros2_control_joint joint_name="leg3_femur_joint"/>
-    <xacro:ros2_control_joint joint_name="leg3_tibia_joint"/>
-    <xacro:ros2_control_joint joint_name="leg4_coxa_joint"/>
-    <xacro:ros2_control_joint joint_name="leg4_femur_joint"/>
-    <xacro:ros2_control_joint joint_name="leg4_tibia_joint"/>
-    <xacro:ros2_control_joint joint_name="leg5_coxa_joint"/>
-    <xacro:ros2_control_joint joint_name="leg5_femur_joint"/>
-    <xacro:ros2_control_joint joint_name="leg5_tibia_joint"/>
-    <xacro:ros2_control_joint joint_name="leg6_coxa_joint"/>
-    <xacro:ros2_control_joint joint_name="leg6_femur_joint"/>
-    <xacro:ros2_control_joint joint_name="leg6_tibia_joint"/>
-  </ros2_control>
+  <xacro:include filename="$(find hexapod_description)/urdf/hexapod.ros2_control.xacro"/>
+  <xacro:hexapod_ros2_control hardware="gazebo"/>
   <gazebo>
     <plugin name="gz_ros2_control::GazeboSimROS2ControlPlugin" filename="libgz_ros2_control-system.so">

Commit message: Make /cmd_vel real m/s and scale the gamepad to the true top speed
The tripod gait walked at 0.6x the commanded speed and ripple/wave had no
fixed relationship, while get_capabilities reported a 0.2 m/s maximum
the robot never reached.

- Plan each phase from the commanded velocity: stance feet move back at
  body speed, swing feet land ahead of neutral by half the stroke
- Shorten phases once the stride hits MAX_STRIDE_LENGTH, down to a new
  min_phase_duration (0.7 s), and cap commands at the gait's top speed
- Report the current gait's real top speeds from get_capabilities
- controller_teleop scales the sticks by those speeds and fetches them
  asynchronously instead of blocking at startup
- Set URDF joint limits to the ST3215's 4.7 rad/s and 2.94 N·m

Co-Authored-By: Claude Opus 5.5 <noreply@anthropic.com>

File: hexapod_ws/src/hexapod_description/urdf/hexapod.urdf.xacro (robot description, xacro)
@@ -1,4 +1,7 @@
 <robot xmlns:xacro="http://ros.org/wiki/xacro" name="hexapod">
   <xacro:arg name="controllers_file" default=""/>
+  <!-- Waveshare ST3215 at 12 V: 2.94 N·m stall torque, 0.222 s/60° no-load speed -->
+  <xacro:property name="servo_effort" value="2.94"/>
+  <xacro:property name="servo_velocity" value="4.7"/>
   <!-- ros2_control hardware: gazebo, mock or st3215 (see hexapod.ros2_control.xacro) -->
   <xacro:arg name="hardware" default="mock"/>
@@ -107,5 +110,5 @@
     <origin xyz="${x_offset} ${y_offset} 0" rpy="0 0 ${yaw}"/>
     <axis xyz="0 0 1"/>
-    <limit lower="-1.57" upper="1.57" effort="1" velocity="1"/>
+    <limit lower="-1.57" upper="1.57" effort="${servo_effort}" velocity="${servo_velocity}"/>
   </joint>
   <!-- FEMUR JOINT -->
@@ -115,5 +118,5 @@
     <origin xyz="${coxa_length} 0 ${femur_z_offset}" rpy="0 0 0"/>
     <axis xyz="0 1 0"/>
-    <limit lower="-1.57" upper="1.57" effort="1" velocity="1"/>
+    <limit lower="-1.57" upper="1.57" effort="${servo_effort}" velocity="${servo_velocity}"/>
   </joint>
   <!-- TIBIA JOINT -->
@@ -123,5 +126,5 @@
     <origin xyz="${femur_length} 0 0" rpy="0 1.5708 0"/>
     <axis xyz="0 1 0"/>
-    <limit lower="-1.57" upper="1.57" effort="1" velocity="1"/>
+    <limit lower="-1.57" upper="1.57" effort="${servo_effort}" velocity="${servo_velocity}"/>
   </joint>
   <!-- COXA TRANSMISSION -->

Commit message: Switch the body frame to REP 103 (+x forward, +y left)
The URDF had +y forward and +x right, which tools like Nav2 and
robot_localization would misread.

- Rotate the body frame -90° in both URDFs: leg offsets, coxa yaws,
  camera mounts and body box rotated with it; leg frames are unchanged,
  so IK and joint angles are unaffected
- Correct the leg comments: legs 1-3 are right (front, middle, rear),
  4-6 left (rear, middle, front)
- FrameConverter stores each leg's URDF yaw and offset instead of a
  mounting angle plus a mirrored flag that didn't match legs 4-6
- MotionIntent uses left (= linear.y) instead of lateral, removing the
  sign flip in strafe mode
- Update unit tests, the sim direction check and the README

Co-Authored-By: Claude Opus 5.5 <noreply@anthropic.com>

File: hexapod_ws/src/hexapod_description/urdf/hexapod.urdf.xacro (robot description, xacro)
@@ -23,4 +23,6 @@
   <link name="base_link">
     <visual>
+      <!-- The body mesh was modelled with +y forward -->
+      <origin xyz="0 0 0" rpy="0 0 -1.5708"/>
       <geometry>
         <mesh filename="package://hexapod_description/meshes/body.dae" scale="1 1 1"/>
@@ -29,4 +31,6 @@
     </visual>
     <collision>
+      <!-- The body mesh was modelled with +y forward -->
+      <origin xyz="0 0 0" rpy="0 0 -1.5708"/>
       <geometry>
         <mesh filename="package://hexapod_description/meshes/body.dae" scale="1 1 1"/>
@@ -163,16 +167,17 @@
 </xacro:macro>
   <!-- ================= LEGS ================= -->
+  <!-- Body frame follows REP 103: +x forward, +y left, +z up -->
+  <!-- Front right -->
+  <xacro:leg name="leg1" x_offset="0.0846" y_offset="-0.06733" yaw="-1.0472" colour="red"/>
+  <!-- Middle right -->
+  <xacro:leg name="leg2" x_offset="0" y_offset="-0.090" yaw="-1.5708" colour="green"/>
+  <!-- Rear right -->
+  <xacro:leg name="leg3" x_offset="-0.0846" y_offset="-0.06733" yaw="-2.0944" colour="blue"/>
+  <!-- Rear left -->
+  <xacro:leg name="leg4" x_offset="-0.0846" y_offset="0.06733" yaw="2.0944" colour="yellow"/>
+  <!-- Middle left -->
+  <xacro:leg name="leg5" x_offset="0" y_offset="0.090" yaw="1.5708" colour="cyan"/>
   <!-- Front left -->
-  <xacro:leg name="leg1" x_offset="0.06733" y_offset="0.0846" yaw="0.5236" colour="red"/>
-  <!-- Middle left -->
-  <xacro:leg name="leg2" x_offset="0.090" y_offset="0" yaw="0" colour="green"/>
-  <!-- Rear left -->
-  <xacro:leg name="leg3" x_offset="0.06733" y_offset="-0.0846" yaw="-0.5236" colour="blue"/>
-  <!-- Front right -->
-  <xacro:leg name="leg4" x_offset="-0.06733" y_offset="-0.0846" yaw="-2.61799" colour="yellow"/>
-  <!-- Middle right -->
-  <xacro:leg name="leg5" x_offset="-0.090" y_offset="0" yaw="-3.14159" colour="cyan"/>
-  <!-- Rear right -->
-  <xacro:leg name="leg6" x_offset="-0.06733" y_offset="0.0846" yaw="2.61799" colour="magenta"/>
+  <xacro:leg name="leg6" x_offset="0.0846" y_offset="0.06733" yaw="1.0472" colour="magenta"/>
   <!-- ================= IMU ================= -->
   <link name="imu_link"/>

File: hexapod_ws/src/hexapod_description/urdf/hexapod_primitives.urdf.xacro (robot description, xacro)
@@ -31,5 +31,5 @@
     <visual>
       <geometry>
-        <box size="0.18 0.17 0.05"/>
+        <box size="0.17 0.18 0.05"/>
       </geometry>
       <material name="black"/>
@@ -37,5 +37,5 @@
     <collision>
       <geometry>
-        <box size="0.18 0.17 0.05"/>
+        <box size="0.17 0.18 0.05"/>
       </geometry>
     </collision>
@@ -182,16 +182,17 @@
 </xacro:macro>
   <!-- ================= LEGS ================= -->
+  <!-- Body frame follows REP 103: +x forward, +y left, +z up -->
+  <!-- Front right -->
+  <xacro:leg name="leg1" x_offset="0.0846" y_offset="-0.06733" yaw="-1.0472" colour="red"/>
+  <!-- Middle right -->
+  <xacro:leg name="leg2" x_offset="0" y_offset="-0.090" yaw="-1.5708" colour="green"/>
+  <!-- Rear right -->
+  <xacro:leg name="leg3" x_offset="-0.0846" y_offset="-0.06733" yaw="-2.0944" colour="blue"/>
+  <!-- Rear left -->
+  <xacro:leg name="leg4" x_offset="-0.0846" y_offset="0.06733" yaw="2.0944" colour="yellow"/>
+  <!-- Middle left -->
+  <xacro:leg name="leg5" x_offset="0" y_offset="0.090" yaw="1.5708" colour="cyan"/>
   <!-- Front left -->
-  <xacro:leg name="leg1" x_offset="0.06733" y_offset="0.0846" yaw="0.5236" colour="red"/>
-  <!-- Middle left -->
-  <xacro:leg name="leg2" x_offset="0.090" y_offset="0" yaw="0" colour="green"/>
-  <!-- Rear left -->
-  <xacro:leg name="leg3" x_offset="0.06733" y_offset="-0.0846" yaw="-0.5236" colour="blue"/>
-  <!-- Front right -->
-  <xacro:leg name="leg4" x_offset="-0.06733" y_offset="-0.0846" yaw="-2.61799" colour="yellow"/>
-  <!-- Middle right -->
-  <xacro:leg name="leg5" x_offset="-0.090" y_offset="0" yaw="-3.14159" colour="cyan"/>
-  <!-- Rear right -->
-  <xacro:leg name="leg6" x_offset="-0.06733" y_offset="0.0846" yaw="2.61799" colour="magenta"/>
+  <xacro:leg name="leg6" x_offset="0.0846" y_offset="0.06733" yaw="1.0472" colour="magenta"/>
   <!-- ================= SENSORS ================= -->
   <link name="camera_link">
@@ -211,5 +212,5 @@
     <parent link="base_link"/>
     <child link="camera_link"/>
-    <origin xyz="0.0 0.0846 0" rpy="0 0 1.5708"/>
+    <origin xyz="0.0846 0.0 0" rpy="0 0 0"/>
   </joint>
   <gazebo reference="camera_link">
@@ -249,5 +250,5 @@
   <parent link="base_link"/>
   <child link="front_depth_camera_link"/>
-  <origin xyz="0.0 0.0846 0.02" rpy="0 0 1.5708"/>
+  <origin xyz="0.0846 0.0 0.02" rpy="0 0 0"/>
 </joint>
 <gazebo reference="front_depth_camera_link">

Commit message: Add RPLIDAR A2M12 support and match the simulated lidar to it
- Run Slamtec's rplidar_ros driver with the other sensors on the real
  robot (256000 baud, lidar_link, published on /lidar/scan like the sim)
- Add a udev rule naming the lidar /dev/rplidar, and bind-mount the Pi's
  /dev into the robot container so the symlink and hot-plugged devices
  are visible
- Share the lidar mount between the real and Gazebo URDFs in
  hexapod.lidar.xacro, so one lidar_z change moves both
- Simulated lidar now matches the A2M12: 10 Hz, 1600 points (0.225 deg),
  0.2-12 m

Co-Authored-By: Claude Opus 5.5 <noreply@anthropic.com>

File: hexapod_ws/src/hexapod_description/urdf/hexapod.urdf.xacro (robot description, xacro)
@@ -187,4 +187,7 @@
     <origin xyz="0.0 0.0 0.03" rpy="0 0 0"/>
   </joint>
+  <!-- ================= LIDAR ================= -->
+  <xacro:include filename="$(find hexapod_description)/urdf/hexapod.lidar.xacro"/>
+  <xacro:hexapod_lidar/>
   <!-- ================= ROS2 CONTROL ================= -->
   <xacro:include filename="$(find hexapod_description)/urdf/hexapod.ros2_control.xacro"/>

File: hexapod_ws/src/hexapod_description/urdf/hexapod_primitives.urdf.xacro (robot description, xacro)
@@ -321,30 +321,15 @@
   </sensor>
 </gazebo>
-<link name="lidar_link">
-  <visual>
-    <geometry><cylinder length="0.04" radius="0.025"/></geometry>
-    <material name="black"/>
-  </visual>
-  <collision>
-    <geometry><cylinder length="0.04" radius="0.025"/></geometry>
-  </collision>
-  <inertial>
-    <mass value="0.1"/>
-    <inertia ixx="0.001" ixy="0" ixz="0" iyy="0.001" iyz="0" izz="0.001"/>
-  </inertial>
-</link>
-<joint name="lidar_joint" type="fixed">
-  <parent link="base_link"/>
-  <child link="lidar_link"/>
-  <origin xyz="0 0 0.05" rpy="0 0 0"/>  <!-- top of body -->
-</joint>
+<xacro:include filename="$(find hexapod_description)/urdf/hexapod.lidar.xacro"/>
+<xacro:hexapod_lidar/>
 <gazebo reference="lidar_link">
   <sensor name="lidar" type="gpu_lidar">
     <always_on>true</always_on>
-    <update_rate>20</update_rate>
+    <!-- RPLIDAR A2M12: 10 Hz, 16 kHz sampling (0.225 deg steps), 0.2-12 m -->
+    <update_rate>10</update_rate>
     <lidar>
       <scan>
         <horizontal>
-          <samples>800</samples>
+          <samples>1600</samples>
           <resolution>1</resolution>
           <min_angle>-3.14159</min_angle>

Commit message: Use the ToF depth camera for low obstacles, add base_footprint, face forwards
Cameras:
- Add hexapod.cameras.xacro, shared by the real and Gazebo models: the
  Arducam ToF camera (B0410) below the Pi Camera Module 3, front facing,
  ToF tilted 10 deg down. The simulated sensors match them (ToF 240x180,
  58.5 deg HFOV, 4 m far mode; Cam 3 standard lens, 66 deg)

Floor frame:
- gait_controller publishes base_footprint -> base_link (the body height,
  republished on set_height); odometry, SLAM and Nav2 use base_footprint,
  so z = 0 in odom is the floor

Nav2:
- Both costmaps take the depth cloud (3-35 cm above the floor, ignoring
  points within 0.3 m of the camera) as 3D voxel layers, so the lidar
  passing over low obstacles doesn't clear what the camera marked
- Global costmap is a 20 x 20 m rolling window: resizing to the growing
  SLAM map wiped the obstacle layer, so low obstacles vanished once the
  camera looked away
- MPPI keeps the Omni model but prefers facing along the path
  (PathAngleCritic forward mode, PreferForwardCritic), so the camera sees
  where the robot walks. Walking backwards into unseen low obstacles had
  got it stuck and drifted the odometry past what SLAM could correct

Add the low_obstacles test world (walled room, 6/10/12/20 cm objects).
Nav2 went through it and back, at least 0.51 m from every object, ending
1-9 cm from the goals.

Co-Authored-By: Claude Opus 5.5 <noreply@anthropic.com>

File: hexapod_ws/src/hexapod_description/urdf/hexapod.urdf.xacro (robot description, xacro)
@@ -190,4 +190,7 @@
   <xacro:include filename="$(find hexapod_description)/urdf/hexapod.lidar.xacro"/>
   <xacro:hexapod_lidar/>
+  <!-- ================= CAMERAS ================= -->
+  <xacro:include filename="$(find hexapod_description)/urdf/hexapod.cameras.xacro"/>
+  <xacro:hexapod_cameras/>
   <!-- ================= ROS2 CONTROL ================= -->
   <xacro:include filename="$(find hexapod_description)/urdf/hexapod.ros2_control.xacro"/>

File: hexapod_ws/src/hexapod_description/urdf/hexapod_primitives.urdf.xacro (robot description, xacro)
@@ -196,31 +196,13 @@
   <xacro:leg name="leg6" x_offset="0.0846" y_offset="0.06733" yaw="1.0472" colour="magenta"/>
   <!-- ================= SENSORS ================= -->
-  <link name="camera_link">
-    <visual>
-      <geometry><box size="0.02 0.05 0"/></geometry>
-      <material name="black"/>
-    </visual>
-    <collision>
-      <geometry><box size="0.02 0.05 0.02"/></geometry>
-    </collision>
-    <inertial>
-      <mass value="0.1"/>
-      <inertia ixx="0.001" ixy="0.0" ixz="0.0" iyy="0.001" iyz="0.0" izz="0.001"/>
-    </inertial>
-  </link>
-  <joint name="camera_joint" type="fixed">
-    <parent link="base_link"/>
-    <child link="camera_link"/>
-    <origin xyz="0.0846 0.0 0" rpy="0 0 0"/>
-  </joint>
   <gazebo reference="camera_link">
   <sensor name="camera" type="camera">
     <always_on>true</always_on>
-    <update_rate>30</update_rate>
+    <update_rate>15</update_rate>
     <camera>
-      <horizontal_fov>1.047</horizontal_fov>  <!-- 60 degrees -->
+      <horizontal_fov>1.152</horizontal_fov>  <!-- Pi Camera Module 3 standard lens: 66 deg -->
       <image>
         <width>640</width>
-        <height>480</height>
+        <height>360</height>
         <format>R8G8B8</format>
       </image>
@@ -234,22 +216,4 @@
   </sensor>
 </gazebo>
-<link name="front_depth_camera_link">
-  <visual>
-    <geometry><box size="0.03 0.03 0.02"/></geometry>
-    <material name="black"/>
-  </visual>
-  <collision>
-    <geometry><box size="0.03 0.03 0.02"/></geometry>
-  </collision>
-  <inertial>
-    <mass value="0.08"/>
-    <inertia ixx="0.0005" ixy="0.0" ixz="0.0" iyy="0.0005" iyz="0.0" izz="0.0005"/>
-  </inertial>
-</link>
-<joint name="front_depth_camera_joint" type="fixed">
-  <parent link="base_link"/>
-  <child link="front_depth_camera_link"/>
-  <origin xyz="0.0846 0.0 0.02" rpy="0 0 0"/>
-</joint>
 <gazebo reference="front_depth_camera_link">
   <sensor name="front_depth_camera" type="depth_camera">
@@ -257,5 +221,5 @@
     <update_rate>$(arg front_depth_rate)</update_rate>
     <camera>
-      <horizontal_fov>1.2043</horizontal_fov>
+      <horizontal_fov>1.021</horizontal_fov>  <!-- Arducam ToF: 70 deg diagonal = 58.5 deg horizontal -->
       <image>
         <width>$(arg front_depth_width)</width>
@@ -264,6 +228,6 @@
       </image>
       <clip>
-        <near>0.2</near>
-        <far>10.0</far>
+        <near>0.1</near>
+        <far>4.0</far>    <!-- far mode -->
       </clip>
     </camera>
@@ -323,4 +287,6 @@
 <xacro:include filename="$(find hexapod_description)/urdf/hexapod.lidar.xacro"/>
 <xacro:hexapod_lidar/>
+<xacro:include filename="$(find hexapod_description)/urdf/hexapod.cameras.xacro"/>
+<xacro:hexapod_cameras/>
 <gazebo reference="lidar_link">
   <sensor name="lidar" type="gpu_lidar">
