Commit message: Widen the femur's range to what the V6.1 CAD allows
The +-1.57 rad joint limits came from the old 180 degree servos; the
ST3215s turn a full circle, so the limits now come from where the
meshes collide. Sweeping the femur against the CAD meshes, raising it
hits the coxa bracket at -100 degrees, and lowering it with the knee
folded puts the tibia into the body at +86 degrees. The femur's limits
are now -1.6 to +1.4 rad (about 10 degrees inside contact) in both
URDFs, and reachable() uses the same range instead of +-1.4.

The coxa and tibia are unchanged. The tibia's bracket hits the femur's
knee servo at a +28 degree fold in the CAD, inside what the gait uses
(+22 standing, up to +77 mid-step), so the knee is being redesigned
before its limit is set.

Co-Authored-By: Claude Opus 5.5 <noreply@anthropic.com>

File: hexapod_ws/src/hexapod_description/urdf/hexapod.urdf.xacro (robot description, xacro)
@@ -4,4 +4,8 @@
   <xacro:property name="servo_effort" value="2.94"/>
   <xacro:property name="servo_velocity" value="4.7"/>
+  <!-- Femur range from the CAD meshes: raising it hits the coxa bracket at -100 deg, lowering it
+       with the knee folded puts the tibia into the body at +86 deg. Both ~10 deg inside contact. -->
+  <xacro:property name="femur_lower" value="-1.6"/>
+  <xacro:property name="femur_upper" value="1.4"/>
   <!-- ros2_control hardware: gazebo, mock or st3215 (see hexapod.ros2_control.xacro) -->
   <xacro:arg name="hardware" default="mock"/>
@@ -121,5 +125,5 @@
     <origin xyz="${coxa_length} 0 0" rpy="0 0 0"/>
     <axis xyz="0 1 0"/>
-    <limit lower="-1.57" upper="1.57" effort="${servo_effort}" velocity="${servo_velocity}"/>
+    <limit lower="${femur_lower}" upper="${femur_upper}" effort="${servo_effort}" velocity="${servo_velocity}"/>
   </joint>
   <!-- TIBIA JOINT -->

File: hexapod_ws/src/hexapod_description/urdf/hexapod_primitives.urdf.xacro (robot description, xacro)
@@ -4,4 +4,8 @@
   <xacro:property name="servo_effort" value="2.94"/>
   <xacro:property name="servo_velocity" value="4.7"/>
+  <!-- Femur range from the CAD meshes: raising it hits the coxa bracket at -100 deg, lowering it
+       with the knee folded puts the tibia into the body at +86 deg. Both ~10 deg inside contact. -->
+  <xacro:property name="femur_lower" value="-1.6"/>
+  <xacro:property name="femur_upper" value="1.4"/>
   <xacro:arg name="front_depth_width" default="640"/>
   <xacro:arg name="front_depth_height" default="480"/>
@@ -145,5 +149,5 @@
     <origin xyz="${coxa_length} 0 0" rpy="0 0 0"/>
     <axis xyz="0 1 0"/>
-    <limit lower="-1.57" upper="1.57" effort="${servo_effort}" velocity="${servo_velocity}"/>
+    <limit lower="${femur_lower}" upper="${femur_upper}" effort="${servo_effort}" velocity="${servo_velocity}"/>
   </joint>
   <!-- TIBIA JOINT -->

Commit message: Limit the knee to the revised V6.1 tibia and keep swings inside it
Sweeping the revised knee in Hexapod_V6.1.step against its meshes,
folding the tibia meets the femur at +60 degrees (39 mm from the knee
axis, so the same whether the shank's piston is in or out), and
straightening at -140. The tibia's limits are now -2.2 to +0.94 rad in
both URDFs and in reachable().

In Gazebo the gait asked for more than that: strafing's middle-leg
swings reach nearly full lift while the foot is still ~40 mm inside
neutral, folding the knee to +55 degrees, and strafing diagonally while
turning once asked for +72 at the knee and -100 at the femur, past the
CAD's contact at both. limitSwingLift() lowers a swinging foot, by
bisection on its height above the swing's ground line, until every
joint is in range with walk leveling applied. Walking and
return-to-start swings (so sitting too) both use it.

Re-run in Gazebo: no commanded angle passes a limit (knee peaks at
+53.9, femur at -84.5), forward walking is unchanged (+53.2 at the
knee, 0.67 m in 6 s), strafing covers the same ground as before, and
the robot still sits and stands.

Co-Authored-By: Claude Opus 5.5 <noreply@anthropic.com>

File: hexapod_ws/src/hexapod_description/urdf/hexapod.urdf.xacro (robot description, xacro)
@@ -8,4 +8,10 @@
   <xacro:property name="femur_lower" value="-1.6"/>
   <xacro:property name="femur_upper" value="1.4"/>
+  <!-- Tibia range from the revised knee in Hexapod_V6.1.step: folding, the tibia meets the femur at
+       +60 deg (whether the shank's piston is in or out); straightening, at -140 deg. Folding keeps
+       ~6 deg in hand. Walking forward peaks at +53 deg; the gait controller lowers any swing that
+       would fold further (limitSwingLift), as strafing's middle-leg swings do. -->
+  <xacro:property name="tibia_lower" value="-2.2"/>
+  <xacro:property name="tibia_upper" value="0.94"/>
   <!-- ros2_control hardware: gazebo, mock or st3215 (see hexapod.ros2_control.xacro) -->
   <xacro:arg name="hardware" default="mock"/>
@@ -133,5 +139,5 @@
     <origin xyz="${femur_length} 0 0" rpy="0 1.5708 0"/>
     <axis xyz="0 1 0"/>
-    <limit lower="-1.57" upper="1.57" effort="${servo_effort}" velocity="${servo_velocity}"/>
+    <limit lower="${tibia_lower}" upper="${tibia_upper}" effort="${servo_effort}" velocity="${servo_velocity}"/>
   </joint>
   <!-- COXA TRANSMISSION -->

File: hexapod_ws/src/hexapod_description/urdf/hexapod_primitives.urdf.xacro (robot description, xacro)
@@ -8,4 +8,10 @@
   <xacro:property name="femur_lower" value="-1.6"/>
   <xacro:property name="femur_upper" value="1.4"/>
+  <!-- Tibia range from the revised knee in Hexapod_V6.1.step: folding, the tibia meets the femur at
+       +60 deg (whether the shank's piston is in or out); straightening, at -140 deg. Folding keeps
+       ~6 deg in hand. Walking forward peaks at +53 deg; the gait controller lowers any swing that
+       would fold further (limitSwingLift), as strafing's middle-leg swings do. -->
+  <xacro:property name="tibia_lower" value="-2.2"/>
+  <xacro:property name="tibia_upper" value="0.94"/>
   <xacro:arg name="front_depth_width" default="640"/>
   <xacro:arg name="front_depth_height" default="480"/>
@@ -157,5 +163,5 @@
     <origin xyz="${femur_length} 0 0" rpy="0 1.5708 0"/>
     <axis xyz="0 1 0"/>
-    <limit lower="-1.57" upper="1.57" effort="${servo_effort}" velocity="${servo_velocity}"/>
+    <limit lower="${tibia_lower}" upper="${tibia_upper}" effort="${servo_effort}" velocity="${servo_velocity}"/>
   </joint>
   <!-- COXA TRANSMISSION -->

Commit message: Widen the knee's range to the lighter V6.1 tibia and update its meshes
Sweeping the new tibia (Hexapod_V6_1_posed.step) against the femur, the
tibia shell meets the femur's at +67.6 degrees folding and -149.8
straightening, both about 100 mm from the knee axis and within a degree
wherever the shank's piston sits; the RM leg agrees. Keeping the old
margins (~6 degrees folding, ~14 straightening), the knee's limits go
from -2.2..+0.94 to -2.35..+1.06 rad in both URDFs and in reachable().
The femur's contacts are unchanged, so its limits stay.

The femur and tibia meshes are re-exported in the same link frames and
detail as before (re-exporting the Oct 16 CAD this way reproduces the
old STLs to ~0.25 mm), with the shank placed so the foot bottom stays at
tibia_length.

In Gazebo nothing is commanded past a limit. Walking forward is
unchanged (knee +53.2, 0.78 m in 6 s); strafing's middle-leg swings now
reach +60.2 instead of being held at +53.9 (same distance covered), and
the diagonal strafe-and-turn peaks at +51.8. The robot sits and stands.
Of the 17 scenarios none fail; the 5 warnings appear the same with the
old limits.

Co-Authored-By: Claude Opus 5.5 <noreply@anthropic.com>

File: hexapod_ws/src/hexapod_description/urdf/hexapod.urdf.xacro (robot description, xacro)
@@ -8,10 +8,10 @@
   <xacro:property name="femur_lower" value="-1.6"/>
   <xacro:property name="femur_upper" value="1.4"/>
-  <!-- Tibia range from the revised knee in Hexapod_V6.1.step: folding, the tibia meets the femur at
-       +60 deg (whether the shank's piston is in or out); straightening, at -140 deg. Folding keeps
-       ~6 deg in hand. Walking forward peaks at +53 deg; the gait controller lowers any swing that
-       would fold further (limitSwingLift), as strafing's middle-leg swings do. -->
-  <xacro:property name="tibia_lower" value="-2.2"/>
-  <xacro:property name="tibia_upper" value="0.94"/>
+  <!-- Tibia range from the lighter V6.1 tibia (Hexapod_V6_1_posed.step): folding, the tibia meets the
+       femur's shell at +67 deg; straightening, at -149 deg (both within a degree wherever the shank's
+       piston sits). Folding keeps ~6 deg in hand and straightening ~14, as before. The gait
+       controller lowers any swing that would fold further (limitSwingLift). -->
+  <xacro:property name="tibia_lower" value="-2.35"/>
+  <xacro:property name="tibia_upper" value="1.06"/>
   <!-- ros2_control hardware: gazebo, mock or st3215 (see hexapod.ros2_control.xacro) -->
   <xacro:arg name="hardware" default="mock"/>
@@ -28,5 +28,6 @@
   <xacro:property name="leg_radius" value="0.148"/>
   <xacro:property name="corner_offset" value="${leg_radius * cos(pi / 4)}"/>
-  <!-- Meshes are exported from the STEP in mm, already in each link's frame -->
+  <!-- Meshes are exported from the STEP in mm, already in each link's frame. The tibia's shank sits
+       where tibia_length assumes, its foot ball 171.9 mm from the knee. -->
   <xacro:property name="mesh_scale" value="0.001 0.001 0.001"/>
   <!-- ================= MATERIALS ================= -->

File: hexapod_ws/src/hexapod_description/urdf/hexapod_primitives.urdf.xacro (robot description, xacro)
@@ -8,10 +8,10 @@
   <xacro:property name="femur_lower" value="-1.6"/>
   <xacro:property name="femur_upper" value="1.4"/>
-  <!-- Tibia range from the revised knee in Hexapod_V6.1.step: folding, the tibia meets the femur at
-       +60 deg (whether the shank's piston is in or out); straightening, at -140 deg. Folding keeps
-       ~6 deg in hand. Walking forward peaks at +53 deg; the gait controller lowers any swing that
-       would fold further (limitSwingLift), as strafing's middle-leg swings do. -->
-  <xacro:property name="tibia_lower" value="-2.2"/>
-  <xacro:property name="tibia_upper" value="0.94"/>
+  <!-- Tibia range from the lighter V6.1 tibia (Hexapod_V6_1_posed.step): folding, the tibia meets the
+       femur's shell at +67 deg; straightening, at -149 deg (both within a degree wherever the shank's
+       piston sits). Folding keeps ~6 deg in hand and straightening ~14, as before. The gait
+       controller lowers any swing that would fold further (limitSwingLift). -->
+  <xacro:property name="tibia_lower" value="-2.35"/>
+  <xacro:property name="tibia_upper" value="1.06"/>
   <xacro:arg name="front_depth_width" default="640"/>
   <xacro:arg name="front_depth_height" default="480"/>
