Commit message: Add slam_toolbox mapping and raise the lidar above the legs
- slam:=true on the simulation and robot launches runs slam_toolbox
  (online async), publishing map -> odom; config based on the package
  defaults, adding scans every 0.2 m / 0.2 rad and using the A2M12 range
- Raise the lidar scan plane from 5 cm to 15 cm above the hip joints. At
  5 cm, 20% of each scan hit the robot's own legs; the knees reach ~12 cm
  (with leg thickness) at the end of a stride
- In the house world, after a 0.6 m square, SLAM was 1.8 cm and 0.2 deg
  from the true pose (odometry alone: 15.5 cm)

Co-Authored-By: Claude Opus 5.5 <noreply@anthropic.com>

File: hexapod_ws/src/hexapod_description/urdf/hexapod.lidar.xacro (robot description, xacro)
@@ -7,5 +7,8 @@
   <xacro:property name="lidar_x" value="0.0"/>
   <xacro:property name="lidar_y" value="0.0"/>
-  <xacro:property name="lidar_z" value="0.05"/>    <!-- above base_link, on top of the body -->
+  <!-- Height of the scan plane above base_link (the hip joint plane). It must clear the legs:
+       the knees reach ~9 cm above the hips at the end of a stride, ~12 cm with the leg's thickness.
+       Below that, the lidar sees the robot's own legs (20% of each scan at 5 cm). -->
+  <xacro:property name="lidar_z" value="0.15"/>
   <xacro:property name="lidar_radius" value="0.038"/>
   <xacro:property name="lidar_height" value="0.041"/>

Commit message: Mount the lidar on the lid and filter out the robot's legs
On the V6.1 body the RPLIDAR sits on the lid, centred, with its scan
plane 73.5 mm above the hip joints instead of on a 15 cm mast, so the
legs cross the scan plane. A laser_filters chain drops returns nearer
than 0.30 m (inside the legs' reach) as NaN and publishes
/lidar/scan_filtered, which SLAM and Nav2 now use. It runs in both the
robot and simulation launches.

In simulation the legs take none of the scan standing, 3% walking (10.5%
at worst) and 5.7% walking with the body at 8 cm; none leak through the
filter, and slam_toolbox maps normally.

Co-Authored-By: Claude Opus 5.5 <noreply@anthropic.com>

File: hexapod_ws/src/hexapod_description/urdf/hexapod.lidar.xacro (robot description, xacro)
@@ -3,12 +3,14 @@
   <!--
     RPLIDAR A2M12 mount, shared by the real and Gazebo models so they stay in the same place.
-    Change lidar_z when the new body is designed.
+    Placed as on the V6.1 body (Hexapod_V6.1.step).
   -->
   <xacro:property name="lidar_x" value="0.0"/>
   <xacro:property name="lidar_y" value="0.0"/>
-  <!-- Height of the scan plane above base_link (the hip joint plane). It must clear the legs:
-       the knees reach ~9 cm above the hips at the end of a stride, ~12 cm with the leg's thickness.
-       Below that, the lidar sees the robot's own legs (20% of each scan at 5 cm). -->
-  <xacro:property name="lidar_z" value="0.15"/>
+  <!-- Height of the scan plane above base_link (the hip joint plane). On the V6.1 body the lidar
+       sits on the lid, centred: lid top 72 mm and hip axis 27.5 mm above the body's base, and the
+       A2M12's scan plane 29 mm above its own base: 73.5 mm. The legs cross it (the
+       knees reach ~9 cm above the hips), so hexapod_bringup's laser_filters.yaml drops everything
+       within 0.30 m and SLAM and Nav2 use /lidar/scan_filtered. -->
+  <xacro:property name="lidar_z" value="0.0735"/>
   <xacro:property name="lidar_radius" value="0.038"/>
   <xacro:property name="lidar_height" value="0.041"/>
