Commit message: Match the URDF and kinematics to the V6.1 design
Dimensions measured from Hexapod_V6.1_stand.step and checked against
the walk pose: coxa 63 mm, femur 100 mm, and the curved tibia's
straight line from knee to the bottom of the foot 186 mm. The coxa
axes are 148 mm from the centre with the corner legs at 45 degrees,
and the femur axes are level with the hips. The solver and the URDF
had different lengths before; both now use these.

New STL meshes are exported from the STEP in each link's frame, with
left and right legs (mirror images) separate, leaving out parts hidden
inside the body and the servos. The Gazebo model uses them as visuals
while keeping simple collision shapes. The lidar and cameras are moved
to the lid and camera pod; the ToF camera is level, as in the pod.

The neutral stance is the CAD stand pose: each foot 0.177 m straight
out and 0.134 m below the hips. Feet now reach ~0.325 m from the
centre, so Nav2's robot_radius goes to 0.39 m and the lidar leg filter
to 0.38 m, and RViz shows the filtered scan. Walk leveling now moves
the feet up to 9 mm sideways, so the clearance test allows for that.
test_kinematics checks IK against both CAD poses.

Servo offsets are unchanged and still need calibrating to these joint
zeros. Not yet run in Gazebo or on the robot.

Co-Authored-By: Claude Opus 5.5 <noreply@anthropic.com>

File: hexapod_ws/src/hexapod_description/urdf/hexapod.cameras.xacro (robot description, xacro)
@@ -6,10 +6,10 @@
       front_depth_camera_link  Arducam ToF camera (B0410): 240x180 depth, 70 deg diagonal FOV, 4 m in far mode
       camera_link              Raspberry Pi Camera Module 3 (standard lens, 66 deg horizontal FOV)
-    The ToF camera tilts down so it sees low obstacles closer to the feet.
+    Placed as in the V6.1 camera pod (Hexapod_V6.1.step), where both face straight ahead.
   -->
-  <xacro:property name="camera_x" value="0.085"/>        <!-- front face of the body -->
-  <xacro:property name="tof_z" value="0.0"/>
-  <xacro:property name="tof_pitch" value="0.1745"/>      <!-- 10 deg down -->
-  <xacro:property name="picam_z" value="0.03"/>
+  <xacro:property name="camera_x" value="0.138"/>        <!-- front of the camera pod -->
+  <xacro:property name="tof_z" value="-0.0124"/>
+  <xacro:property name="tof_pitch" value="0.0"/>
+  <xacro:property name="picam_z" value="0.0257"/>
   <xacro:property name="picam_pitch" value="0.0"/>
   <xacro:macro name="hexapod_cameras">

File: hexapod_ws/src/hexapod_description/urdf/hexapod.lidar.xacro (robot description, xacro)
@@ -8,9 +8,9 @@
   <xacro:property name="lidar_y" value="0.0"/>
   <!-- Height of the scan plane above base_link (the hip joint plane). On the V6.1 body the lidar
-       sits on the lid, centred: lid top 72 mm and hip axis 27.5 mm above the body's base, and the
-       A2M12's scan plane 29 mm above its own base: 73.5 mm. The legs cross it (the
-       knees reach ~9 cm above the hips), so hexapod_bringup's laser_filters.yaml drops everything
-       within 0.30 m and SLAM and Nav2 use /lidar/scan_filtered. -->
-  <xacro:property name="lidar_z" value="0.0735"/>
+       sits on the lid, centred: lid top 72 mm and hip axis 33.85 mm above the body's base, and the
+       A2M12's scan plane 29 mm above its own base: 67 mm. The legs cross it (the top of the
+       tibia is level with it when standing), so hexapod_bringup's laser_filters.yaml drops
+       everything within 0.38 m and SLAM and Nav2 use /lidar/scan_filtered. -->
+  <xacro:property name="lidar_z" value="0.067"/>
   <xacro:property name="lidar_radius" value="0.038"/>
   <xacro:property name="lidar_height" value="0.041"/>

File: hexapod_ws/src/hexapod_description/urdf/hexapod.urdf.xacro (robot description, xacro)
@@ -8,8 +8,16 @@
   <xacro:arg name="serial_port" default="/dev/ttyAMA0"/>
   <!-- ================= CONSTANTS ================= -->
-  <xacro:property name="coxa_length" value="0.0375"/>
-  <xacro:property name="femur_length" value="0.1"/>
-  <xacro:property name="tibia_length" value="0.15"/>
-  <xacro:property name="femur_z_offset" value="0.0106"/>
+  <!-- Measured from Hexapod_V6.1 (joint caps and feet). base_link sits on the hip plane, the
+       height of the femur axes, 33.85 mm above the bottom of the body. -->
+  <xacro:property name="coxa_length" value="0.063"/>    <!-- coxa axis to femur axis, level -->
+  <xacro:property name="femur_length" value="0.1"/>     <!-- femur axis to knee axis -->
+  <!-- Knee axis to the bottom of the foot, along the straight line through the curved tibia
+       (171.95 mm to the foot ball's centre, plus its 14 mm radius) -->
+  <xacro:property name="tibia_length" value="0.186"/>
+  <!-- Coxa axes: 148 mm from the centre, the corner legs at 45 degrees -->
+  <xacro:property name="leg_radius" value="0.148"/>
+  <xacro:property name="corner_offset" value="${leg_radius * cos(pi / 4)}"/>
+  <!-- Meshes are exported from the STEP in mm, already in each link's frame -->
+  <xacro:property name="mesh_scale" value="0.001 0.001 0.001"/>
   <!-- ================= MATERIALS ================= -->
   <material name="black"><color rgba="0.1 0.1 0.1 1"/></material>
@@ -23,16 +31,12 @@
   <link name="base_link">
     <visual>
-      <!-- The body mesh was modelled with +y forward -->
-      <origin xyz="0 0 0" rpy="0 0 -1.5708"/>
-      <geometry>
-        <mesh filename="package://hexapod_description/meshes/body.dae" scale="1 1 1"/>
+      <geometry>
+        <mesh filename="package://hexapod_description/meshes/body.stl" scale="${mesh_scale}"/>
       </geometry>
       <material name="black"/>
     </visual>
     <collision>
-      <!-- The body mesh was modelled with +y forward -->
-      <origin xyz="0 0 0" rpy="0 0 -1.5708"/>
-      <geometry>
-        <mesh filename="package://hexapod_description/meshes/body.dae" scale="1 1 1"/>
+      <geometry>
+        <mesh filename="package://hexapod_description/meshes/body.stl" scale="${mesh_scale}"/>
       </geometry>
     </collision>
@@ -44,18 +48,17 @@
   </link>
 <!-- ================= LEG LINKS ================= -->
-<xacro:macro name="leg" params="name x_offset y_offset yaw colour">
+<!-- side: left or right, the left legs being mirror images of the right -->
+<xacro:macro name="leg" params="name side x_offset y_offset yaw colour">
   <!-- COXA -->
   <link name="${name}_coxa">
     <visual>
-      <origin xyz="0 0 0" rpy="0 0 1.5708"/>
-      <geometry>
-        <mesh filename="package://hexapod_description/meshes/coxa.dae" scale="1 1 1"/>
+      <geometry>
+        <mesh filename="package://hexapod_description/meshes/coxa_${side}.stl" scale="${mesh_scale}"/>
       </geometry>
       <material name="${colour}"/>
     </visual>
     <collision>
-      <origin xyz="0 0 0" rpy="0 0 1.5708"/>
-      <geometry>
-        <mesh filename="package://hexapod_description/meshes/coxa.dae" scale="1 1 1"/>
+      <geometry>
+        <mesh filename="package://hexapod_description/meshes/coxa_${side}.stl" scale="${mesh_scale}"/>
       </geometry>
     </collision>
@@ -69,14 +72,12 @@
   <link name="${name}_femur">
     <visual>
-      <origin xyz="0 0 0" rpy="0 0 1.5708"/>
-      <geometry>
-        <mesh filename="package://hexapod_description/meshes/femur.dae" scale="1 1 1"/>
+      <geometry>
+        <mesh filename="package://hexapod_description/meshes/femur_${side}.stl" scale="${mesh_scale}"/>
       </geometry>
       <material name="${colour}"/>
     </visual>
     <collision>
-      <origin xyz="0 0 0" rpy="0 0 1.5708"/>
-      <geometry>
-        <mesh filename="package://hexapod_description/meshes/femur.dae" scale="1 1 1"/>
+      <geometry>
+        <mesh filename="package://hexapod_description/meshes/femur_${side}.stl" scale="${mesh_scale}"/>
       </geometry>
     </collision>
@@ -90,14 +91,12 @@
   <link name="${name}_tibia">
     <visual>
-      <origin xyz="0 0 0" rpy="0 0 1.5708"/>
-      <geometry>
-        <mesh filename="package://hexapod_description/meshes/tibia.dae" scale="1 1 1"/>
+      <geometry>
+        <mesh filename="package://hexapod_description/meshes/tibia_${side}.stl" scale="${mesh_scale}"/>
       </geometry>
       <material name="${colour}"/>
     </visual>
     <collision>
-      <origin xyz="0 0 0" rpy="0 0 1.5708"/>
-      <geometry>
-        <mesh filename="package://hexapod_description/meshes/tibia.dae" scale="1 1 1"/>
+      <geometry>
+        <mesh filename="package://hexapod_description/meshes/tibia_${side}.stl" scale="${mesh_scale}"/>
       </geometry>
     </collision>
@@ -120,5 +119,5 @@
     <parent link="${name}_coxa"/>
     <child link="${name}_femur"/>
-    <origin xyz="${coxa_length} 0 ${femur_z_offset}" rpy="0 0 0"/>
+    <origin xyz="${coxa_length} 0 0" rpy="0 0 0"/>
     <axis xyz="0 1 0"/>
     <limit lower="-1.57" upper="1.57" effort="${servo_effort}" velocity="${servo_velocity}"/>
@@ -169,15 +168,15 @@
   <!-- Body frame follows REP 103: +x forward, +y left, +z up -->
   <!-- Front right -->
-  <xacro:leg name="leg1" x_offset="0.0846" y_offset="-0.06733" yaw="-1.0472" colour="red"/>
+  <xacro:leg name="leg1" side="right" x_offset="${corner_offset}" y_offset="${-corner_offset}" yaw="${-pi / 4}" colour="red"/>
   <!-- Middle right -->
-  <xacro:leg name="leg2" x_offset="0" y_offset="-0.090" yaw="-1.5708" colour="green"/>
+  <xacro:leg name="leg2" side="right" x_offset="0" y_offset="${-leg_radius}" yaw="${-pi / 2}" colour="green"/>
   <!-- Rear right -->
-  <xacro:leg name="leg3" x_offset="-0.0846" y_offset="-0.06733" yaw="-2.0944" colour="blue"/>
+  <xacro:leg name="leg3" side="right" x_offset="${-corner_offset}" y_offset="${-corner_offset}" yaw="${-3 * pi / 4}" colour="blue"/>
   <!-- Rear left -->
-  <xacro:leg name="leg4" x_offset="-0.0846" y_offset="0.06733" yaw="2.0944" colour="yellow"/>
+  <xacro:leg name="leg4" side="left" x_offset="${-corner_offset}" y_offset="${corner_offset}" yaw="${3 * pi / 4}" colour="yellow"/>
   <!-- Middle left -->
-  <xacro:leg name="leg5" x_offset="0" y_offset="0.090" yaw="1.5708" colour="cyan"/>
+  <xacro:leg name="leg5" side="left" x_offset="0" y_offset="${leg_radius}" yaw="${pi / 2}" colour="cyan"/>
   <!-- Front left -->
-  <xacro:leg name="leg6" x_offset="0.0846" y_offset="0.06733" yaw="1.0472" colour="magenta"/>
+  <xacro:leg name="leg6" side="left" x_offset="${corner_offset}" y_offset="${corner_offset}" yaw="${pi / 4}" colour="magenta"/>
   <!-- ================= IMU ================= -->
   <link name="imu_link"/>

File: hexapod_ws/src/hexapod_description/urdf/hexapod_primitives.urdf.xacro (robot description, xacro)
@@ -8,14 +8,24 @@
   <xacro:arg name="front_depth_rate" default="8"/>
   <!-- ================= CONSTANTS ================= -->
-  <xacro:property name="coxa_length" value="0.055"/>
-  <xacro:property name="femur_length" value="0.09"/>
-  <xacro:property name="tibia_length" value="0.15"/>
-  <xacro:property name="coxa_width" value="0.048"/>
-  <xacro:property name="coxa_height" value="0.06"/>
-  <xacro:property name="femur_radius" value="0.029"/>
-  <xacro:property name="tibia_radius" value="0.0225"/>
+  <!-- Hexapod_V6.1, as in hexapod.urdf.xacro (base_link on the hip plane) -->
+  <xacro:property name="coxa_length" value="0.063"/>
+  <xacro:property name="femur_length" value="0.1"/>
+  <!-- Straight line from the knee to the bottom of the foot; the real tibia curves outwards -->
+  <xacro:property name="tibia_length" value="0.186"/>
+  <xacro:property name="leg_radius" value="0.148"/>
+  <xacro:property name="corner_offset" value="${leg_radius * cos(pi / 4)}"/>
+  <!-- Octagonal body 220 mm across flats, 72 mm tall with the lid, its base 33.85 mm below the hips -->
+  <xacro:property name="body_radius" value="0.11"/>
+  <xacro:property name="body_height" value="0.072"/>
+  <xacro:property name="body_z" value="${body_height / 2 - 0.03385}"/>
+  <xacro:property name="coxa_width" value="0.054"/>
+  <xacro:property name="coxa_height" value="0.045"/>
+  <xacro:property name="femur_radius" value="0.025"/>
+  <xacro:property name="tibia_radius" value="0.017"/>
   <xacro:property name="cscale" value="0.95"/>
+  <!-- Visuals are the real robot's meshes (as in hexapod.urdf.xacro); collisions stay simple shapes -->
+  <xacro:property name="mesh_scale" value="0.001 0.001 0.001"/>
   <!-- Rubber foot at the tibia tip; its bottom sits at tibia_length so the IK leg length is unchanged -->
-  <xacro:property name="foot_radius" value="0.012"/>
+  <xacro:property name="foot_radius" value="0.014"/>
   <xacro:property name="foot_friction" value="1.5"/>
   <!-- ================= MATERIALS ================= -->
@@ -31,11 +41,12 @@
     <visual>
       <geometry>
-        <box size="0.17 0.18 0.05"/>
+        <mesh filename="package://hexapod_description/meshes/body.stl" scale="${mesh_scale}"/>
       </geometry>
       <material name="black"/>
     </visual>
     <collision>
-      <geometry>
-        <box size="0.17 0.18 0.05"/>
+      <origin xyz="0 0 ${body_z}"/>
+      <geometry>
+        <cylinder length="${body_height}" radius="${body_radius}"/>
       </geometry>
     </collision>
@@ -47,11 +58,11 @@
   </link>
 <!-- ================= LEG LINKS ================= -->
-<xacro:macro name="leg" params="name x_offset y_offset yaw colour">
+<!-- side: left or right, the left legs being mirror images of the right -->
+<xacro:macro name="leg" params="name side x_offset y_offset yaw colour">
   <!-- COXA -->
   <link name="${name}_coxa">
     <visual>
-      <origin xyz="${coxa_length/2} 0 0" rpy="0 0 0"/>
-      <geometry>
-        <box size="${coxa_length} ${coxa_width} ${coxa_height}"/>
+      <geometry>
+        <mesh filename="package://hexapod_description/meshes/coxa_${side}.stl" scale="${mesh_scale}"/>
       </geometry>
       <material name="${colour}"/>
@@ -72,8 +83,6 @@
   <link name="${name}_femur">
     <visual>
-      <!-- Cylinder base aligned with joint -->
-      <origin xyz="${femur_length/2} 0 0" rpy="0 -1.5708 0"/>
-      <geometry>
-        <cylinder length="${femur_length}" radius="${femur_radius}"/>
+      <geometry>
+        <mesh filename="package://hexapod_description/meshes/femur_${side}.stl" scale="${mesh_scale}"/>
       </geometry>
       <material name="${colour}"/>
@@ -94,7 +103,6 @@
   <link name="${name}_tibia">
     <visual>
-      <origin xyz="${tibia_length/2} 0 0" rpy="0 -1.5708 0"/>
-      <geometry>
-        <cylinder length="${tibia_length}" radius="${tibia_radius}"/>
+      <geometry>
+        <mesh filename="package://hexapod_description/meshes/tibia_${side}.stl" scale="${mesh_scale}"/>
       </geometry>
       <material name="${colour}"/>
@@ -184,15 +192,15 @@
   <!-- Body frame follows REP 103: +x forward, +y left, +z up -->
   <!-- Front right -->
-  <xacro:leg name="leg1" x_offset="0.0846" y_offset="-0.06733" yaw="-1.0472" colour="red"/>
+  <xacro:leg name="leg1" side="right" x_offset="${corner_offset}" y_offset="${-corner_offset}" yaw="${-pi / 4}" colour="red"/>
   <!-- Middle right -->
-  <xacro:leg name="leg2" x_offset="0" y_offset="-0.090" yaw="-1.5708" colour="green"/>
+  <xacro:leg name="leg2" side="right" x_offset="0" y_offset="${-leg_radius}" yaw="${-pi / 2}" colour="green"/>
   <!-- Rear right -->
-  <xacro:leg name="leg3" x_offset="-0.0846" y_offset="-0.06733" yaw="-2.0944" colour="blue"/>
+  <xacro:leg name="leg3" side="right" x_offset="${-corner_offset}" y_offset="${-corner_offset}" yaw="${-3 * pi / 4}" colour="blue"/>
   <!-- Rear left -->
-  <xacro:leg name="leg4" x_offset="-0.0846" y_offset="0.06733" yaw="2.0944" colour="yellow"/>
+  <xacro:leg name="leg4" side="left" x_offset="${-corner_offset}" y_offset="${corner_offset}" yaw="${3 * pi / 4}" colour="yellow"/>
   <!-- Middle left -->
-  <xacro:leg name="leg5" x_offset="0" y_offset="0.090" yaw="1.5708" colour="cyan"/>
+  <xacro:leg name="leg5" side="left" x_offset="0" y_offset="${leg_radius}" yaw="${pi / 2}" colour="cyan"/>
   <!-- Front left -->
-  <xacro:leg name="leg6" x_offset="0.0846" y_offset="0.06733" yaw="1.0472" colour="magenta"/>
+  <xacro:leg name="leg6" side="left" x_offset="${corner_offset}" y_offset="${corner_offset}" yaw="${pi / 4}" colour="magenta"/>
   <!-- ================= SENSORS ================= -->
   <gazebo reference="camera_link">
