Commit message: Give the URDF real masses and inertias from the V6.1 CAD
Every link had a placeholder inertial: a 1 kg body with 0.1 kg m^2
of inertia and 50-100 g legs, so the simulated robot weighed about
2.2 kg with link inertias 10-1000 times too big. The new
scripts/mass_properties.py reads Hexapod_V6.1.step (the body and one
leg), puts each solid in the link it moves with, and writes
urdf/hexapod.inertials.xacro, which both URDFs now use.

Bought parts get their real weight spread over their CAD volume
(ST3215 55 g, Pi 5 46 g, RPLIDAR A2M12 190 g; the battery, boards and
cameras are estimates). Printed parts are the filament's density
(PA12-CF legs, PETG body, TPU feet) at 60% of solid for walls and
infill, until the parts are weighed and put in MEASURED. The leg's
frames come from the joint caps and the foot ball, and the right legs
mirror the left. The robot comes to 3.32 kg: body 1.11 kg, coxa 93 g,
femur 172 g (two servos), tibia 103 g.

The lidar and camera links are fixed to base_link and merged into it,
so their masses drop to 1 g now that the body's inertial counts them.

Co-Authored-By: Claude Opus 5.5 (1M context) <noreply@anthropic.com>
Claude-Session: https://claude.ai/code/session_0161HQCLwto8ZfvbUyYjHkWJ

File: hexapod_ws/src/hexapod_description/urdf/hexapod.cameras.xacro (robot description, xacro)
@@ -22,7 +22,8 @@
         <geometry><box size="0.01 0.038 0.038"/></geometry>
       </collision>
+      <!-- Its mass is in base_link's inertial (hexapod.inertials.xacro); fixed joints are merged into base_link -->
       <inertial>
-        <mass value="0.02"/>
-        <inertia ixx="0.00001" ixy="0" ixz="0" iyy="0.00001" iyz="0" izz="0.00001"/>
+        <mass value="0.001"/>
+        <inertia ixx="1e-8" ixy="0" ixz="0" iyy="1e-8" iyz="0" izz="1e-8"/>
       </inertial>
     </link>
@@ -40,7 +41,8 @@
         <geometry><box size="0.01 0.025 0.024"/></geometry>
       </collision>
+      <!-- Its mass is in base_link's inertial (hexapod.inertials.xacro); fixed joints are merged into base_link -->
       <inertial>
-        <mass value="0.01"/>
-        <inertia ixx="0.00001" ixy="0" ixz="0" iyy="0.00001" iyz="0" izz="0.00001"/>
+        <mass value="0.001"/>
+        <inertia ixx="1e-8" ixy="0" ixz="0" iyy="1e-8" iyz="0" izz="1e-8"/>
       </inertial>
     </link>

File: hexapod_ws/src/hexapod_description/urdf/hexapod.lidar.xacro (robot description, xacro)
@@ -24,7 +24,8 @@
         <geometry><cylinder length="${lidar_height}" radius="${lidar_radius}"/></geometry>
       </collision>
+      <!-- Its mass is in base_link's inertial (hexapod.inertials.xacro); fixed joints are merged into base_link -->
       <inertial>
-        <mass value="0.19"/>
-        <inertia ixx="0.0001" ixy="0" ixz="0" iyy="0.0001" iyz="0" izz="0.0001"/>
+        <mass value="0.001"/>
+        <inertia ixx="1e-8" ixy="0" ixz="0" iyy="1e-8" iyz="0" izz="1e-8"/>
       </inertial>
     </link>

File: hexapod_ws/src/hexapod_description/urdf/hexapod.urdf.xacro (robot description, xacro)
@@ -31,4 +31,6 @@
        where tibia_length assumes, its foot ball 171.9 mm from the knee. -->
   <xacro:property name="mesh_scale" value="0.001 0.001 0.001"/>
+  <!-- Masses and inertias from the CAD (scripts/mass_properties.py) -->
+  <xacro:include filename="$(find hexapod_description)/urdf/hexapod.inertials.xacro"/>
   <!-- ================= MATERIALS ================= -->
   <material name="black"><color rgba="0.1 0.1 0.1 1"/></material>
@@ -52,9 +54,5 @@
       </geometry>
     </collision>
-    <inertial>
-      <mass value="1.0"/>
-      <origin xyz="0 0 0"/>
-      <inertia ixx="0.1" ixy="0.0" ixz="0.0" iyy="0.1" iyz="0.0" izz="0.1"/>
-    </inertial>
+    <xacro:hexapod_base_inertial/>
   </link>
 <!-- ================= LEG LINKS ================= -->
@@ -74,9 +72,5 @@
       </geometry>
     </collision>
-    <inertial>
-      <mass value="0.1"/>
-      <origin xyz="0 0 0"/>
-      <inertia ixx="0.01" ixy="0.0" ixz="0.0" iyy="0.01" iyz="0.0" izz="0.01"/>
-    </inertial>
+    <xacro:hexapod_leg_inertial link="coxa" side="${side}"/>
   </link>
   <!-- FEMUR -->
@@ -93,9 +87,5 @@
       </geometry>
     </collision>
-    <inertial>
-      <mass value="0.05"/>
-      <origin xyz="0 0 0"/>
-      <inertia ixx="0.001" ixy="0.0" ixz="0.0" iyy="0.001" iyz="0.0" izz="0.001"/>
-    </inertial>
+    <xacro:hexapod_leg_inertial link="femur" side="${side}"/>
   </link>
   <!-- TIBIA -->
@@ -112,9 +102,5 @@
       </geometry>
     </collision>
-    <inertial>
-      <mass value="0.05"/>
-      <origin xyz="0 0 0"/>
-      <inertia ixx="0.001" ixy="0.0" ixz="0.0" iyy="0.001" iyz="0.0" izz="0.001"/>
-    </inertial>
+    <xacro:hexapod_leg_inertial link="tibia" side="${side}"/>
   </link>
   <!-- COXA JOINT -->

File: hexapod_ws/src/hexapod_description/urdf/hexapod_primitives.urdf.xacro (robot description, xacro)
@@ -39,4 +39,6 @@
   <xacro:property name="foot_radius" value="0.014"/>
   <xacro:property name="foot_friction" value="1.5"/>
+  <!-- Masses and inertias from the CAD (scripts/mass_properties.py) -->
+  <xacro:include filename="$(find hexapod_description)/urdf/hexapod.inertials.xacro"/>
   <!-- ================= MATERIALS ================= -->
   <material name="black"><color rgba="0.1 0.1 0.1 1"/></material>
@@ -61,9 +63,5 @@
       </geometry>
     </collision>
-    <inertial>
-      <mass value="1.0"/>
-      <origin xyz="0 0 0"/>
-      <inertia ixx="0.1" ixy="0.0" ixz="0.0" iyy="0.1" iyz="0.0" izz="0.1"/>
-    </inertial>
+    <xacro:hexapod_base_inertial/>
   </link>
 <!-- ================= LEG LINKS ================= -->
@@ -84,9 +82,5 @@
       </geometry>
     </collision>
-    <inertial>
-      <mass value="0.1"/>
-      <origin xyz="${coxa_length/2} 0 0"/>
-      <inertia ixx="0.01" ixy="0.0" ixz="0.0" iyy="0.01" iyz="0.0" izz="0.01"/>
-    </inertial>
+    <xacro:hexapod_leg_inertial link="coxa" side="${side}"/>
   </link>
   <!-- FEMUR -->
@@ -104,9 +98,5 @@
       </geometry>
     </collision>
-    <inertial>
-      <mass value="0.05"/>
-      <origin xyz="${femur_length/2} 0 0"/>
-      <inertia ixx="0.001" ixy="0.0" ixz="0.0" iyy="0.001" iyz="0.0" izz="0.001"/>
-    </inertial>
+    <xacro:hexapod_leg_inertial link="femur" side="${side}"/>
   </link>
   <!-- TIBIA -->
@@ -131,9 +121,5 @@
       </geometry>
     </collision>
-    <inertial>
-      <mass value="0.05"/>
-      <origin xyz="${tibia_length/2} 0 0"/>
-      <inertia ixx="0.001" ixy="0.0" ixz="0.0" iyy="0.001" iyz="0.0" izz="0.001"/>
-    </inertial>
+    <xacro:hexapod_leg_inertial link="tibia" side="${side}"/>
   </link>
   <gazebo reference="${name}_tibia">
@@ -262,7 +248,8 @@
     <geometry><box size="0.015 0.015 0.005"/></geometry>
   </collision>
+  <!-- Its mass is in base_link's inertial (hexapod.inertials.xacro); fixed joints are merged into base_link -->
   <inertial>
-    <mass value="0.01"/>
-    <inertia ixx="1e-6" ixy="0.0" ixz="0.0" iyy="1e-6" iyz="0.0" izz="1e-6"/>
+    <mass value="0.001"/>
+    <inertia ixx="1e-8" ixy="0" ixz="0" iyy="1e-8" iyz="0" izz="1e-8"/>
   </inertial>
 </link>
