Commit message: Move the legs to the slimmer V6.1 body
Hexapod_V6.1.step now has a 220 x 161 mm body. The middle legs' mounts
sit on side faces 80.4 mm from the centre, so their coxa axes are
118.36 mm out instead of 148. The corner legs stay at 45 degrees but
sit in the middle of chamfers centred at (92.32, 62.68) mm, which puts
their coxa axes at (119.16, 89.52) mm. Both URDFs and the gait
controller's FrameConverter use the new positions.

body.stl is re-exported from the new STEP in base_link (the body and
lid shells, lidar, camera pod and six leg mounts), and the primitive
model's body collision becomes a 220 x 161 mm box. The base inertial
is regenerated with the leg mounts in their new places.

The feet still stand out to ~0.325 m at the corners (the middle feet
now ~0.295 m), so Nav2's robot_radius and the lidar leg filter stay.

Co-Authored-By: Claude Opus 5.5 (1M context) <noreply@anthropic.com>
Claude-Session: https://claude.ai/code/session_0161HQCLwto8ZfvbUyYjHkWJ

File: hexapod_ws/src/hexapod_description/urdf/hexapod.inertials.xacro (robot description, xacro)
@@ -7,5 +7,5 @@
       <mass value="1.1082"/>
       <origin xyz="-0.00433 0.00009 0.00993"/>
-      <inertia ixx="3.9990e-03" ixy="-1.1081e-06" ixz="-5.7272e-05" iyy="5.5599e-03" iyz="6.0138e-08" izz="7.5943e-03"/>
+      <inertia ixx="3.4133e-03" ixy="-1.1081e-06" ixz="-5.7272e-05" iyy="5.8450e-03" iyz="6.0138e-08" izz="7.2937e-03"/>
     </inertial>
   </xacro:macro>

File: hexapod_ws/src/hexapod_description/urdf/hexapod.urdf.xacro (robot description, xacro)
@@ -25,7 +25,10 @@
        (171.95 mm to the foot ball's centre, plus its 14 mm radius) -->
   <xacro:property name="tibia_length" value="0.186"/>
-  <!-- Coxa axes: 148 mm from the centre, the corner legs at 45 degrees -->
-  <xacro:property name="leg_radius" value="0.148"/>
-  <xacro:property name="corner_offset" value="${leg_radius * cos(pi / 4)}"/>
+  <!-- Coxa axes on the slimmer V6.1 body (220 x 161 mm). Every leg mount's coxa axis is 37.96 mm
+       out from the body face it sits on: the middle legs' faces are 80.4 mm from the centre, and
+       the corner legs sit in the middle of 45 degree chamfers whose centres are at (92.32, 62.68). -->
+  <xacro:property name="middle_leg_y" value="0.11836"/>
+  <xacro:property name="corner_leg_x" value="0.11916"/>
+  <xacro:property name="corner_leg_y" value="0.08952"/>
   <!-- Meshes are exported from the STEP in mm, already in each link's frame. The tibia's shank sits
        where tibia_length assumes, its foot ball 171.9 mm from the knee. -->
@@ -165,15 +168,15 @@
   <!-- Body frame follows REP 103: +x forward, +y left, +z up -->
   <!-- Front right -->
-  <xacro:leg name="leg1" side="right" x_offset="${corner_offset}" y_offset="${-corner_offset}" yaw="${-pi / 4}" colour="red"/>
+  <xacro:leg name="leg1" side="right" x_offset="${corner_leg_x}" y_offset="${-corner_leg_y}" yaw="${-pi / 4}" colour="red"/>
   <!-- Middle right -->
-  <xacro:leg name="leg2" side="right" x_offset="0" y_offset="${-leg_radius}" yaw="${-pi / 2}" colour="green"/>
+  <xacro:leg name="leg2" side="right" x_offset="0" y_offset="${-middle_leg_y}" yaw="${-pi / 2}" colour="green"/>
   <!-- Rear right -->
-  <xacro:leg name="leg3" side="right" x_offset="${-corner_offset}" y_offset="${-corner_offset}" yaw="${-3 * pi / 4}" colour="blue"/>
+  <xacro:leg name="leg3" side="right" x_offset="${-corner_leg_x}" y_offset="${-corner_leg_y}" yaw="${-3 * pi / 4}" colour="blue"/>
   <!-- Rear left -->
-  <xacro:leg name="leg4" side="left" x_offset="${-corner_offset}" y_offset="${corner_offset}" yaw="${3 * pi / 4}" colour="yellow"/>
+  <xacro:leg name="leg4" side="left" x_offset="${-corner_leg_x}" y_offset="${corner_leg_y}" yaw="${3 * pi / 4}" colour="yellow"/>
   <!-- Middle left -->
-  <xacro:leg name="leg5" side="left" x_offset="0" y_offset="${leg_radius}" yaw="${pi / 2}" colour="cyan"/>
+  <xacro:leg name="leg5" side="left" x_offset="0" y_offset="${middle_leg_y}" yaw="${pi / 2}" colour="cyan"/>
   <!-- Front left -->
-  <xacro:leg name="leg6" side="left" x_offset="${corner_offset}" y_offset="${corner_offset}" yaw="${pi / 4}" colour="magenta"/>
+  <xacro:leg name="leg6" side="left" x_offset="${corner_leg_x}" y_offset="${corner_leg_y}" yaw="${pi / 4}" colour="magenta"/>
   <!-- ================= IMU ================= -->
   <link name="imu_link"/>

File: hexapod_ws/src/hexapod_description/urdf/hexapod_primitives.urdf.xacro (robot description, xacro)
@@ -23,8 +23,10 @@
   <!-- Straight line from the knee to the bottom of the foot; the real tibia curves outwards -->
   <xacro:property name="tibia_length" value="0.186"/>
-  <xacro:property name="leg_radius" value="0.148"/>
-  <xacro:property name="corner_offset" value="${leg_radius * cos(pi / 4)}"/>
-  <!-- Octagonal body 220 mm across flats, 72 mm tall with the lid, its base 33.85 mm below the hips -->
-  <xacro:property name="body_radius" value="0.11"/>
+  <xacro:property name="middle_leg_y" value="0.11836"/>
+  <xacro:property name="corner_leg_x" value="0.11916"/>
+  <xacro:property name="corner_leg_y" value="0.08952"/>
+  <!-- Body 220 mm long and 161 mm wide, 72 mm tall with the lid, its base 33.85 mm below the hips -->
+  <xacro:property name="body_length" value="0.22"/>
+  <xacro:property name="body_width" value="0.161"/>
   <xacro:property name="body_height" value="0.072"/>
   <xacro:property name="body_z" value="${body_height / 2 - 0.03385}"/>
@@ -60,5 +62,5 @@
       <origin xyz="0 0 ${body_z}"/>
       <geometry>
-        <cylinder length="${body_height}" radius="${body_radius}"/>
+        <box size="${body_length} ${body_width} ${body_height}"/>
       </geometry>
     </collision>
@@ -188,15 +190,15 @@
   <!-- Body frame follows REP 103: +x forward, +y left, +z up -->
   <!-- Front right -->
-  <xacro:leg name="leg1" side="right" x_offset="${corner_offset}" y_offset="${-corner_offset}" yaw="${-pi / 4}" colour="red"/>
+  <xacro:leg name="leg1" side="right" x_offset="${corner_leg_x}" y_offset="${-corner_leg_y}" yaw="${-pi / 4}" colour="red"/>
   <!-- Middle right -->
-  <xacro:leg name="leg2" side="right" x_offset="0" y_offset="${-leg_radius}" yaw="${-pi / 2}" colour="green"/>
+  <xacro:leg name="leg2" side="right" x_offset="0" y_offset="${-middle_leg_y}" yaw="${-pi / 2}" colour="green"/>
   <!-- Rear right -->
-  <xacro:leg name="leg3" side="right" x_offset="${-corner_offset}" y_offset="${-corner_offset}" yaw="${-3 * pi / 4}" colour="blue"/>
+  <xacro:leg name="leg3" side="right" x_offset="${-corner_leg_x}" y_offset="${-corner_leg_y}" yaw="${-3 * pi / 4}" colour="blue"/>
   <!-- Rear left -->
-  <xacro:leg name="leg4" side="left" x_offset="${-corner_offset}" y_offset="${corner_offset}" yaw="${3 * pi / 4}" colour="yellow"/>
+  <xacro:leg name="leg4" side="left" x_offset="${-corner_leg_x}" y_offset="${corner_leg_y}" yaw="${3 * pi / 4}" colour="yellow"/>
   <!-- Middle left -->
-  <xacro:leg name="leg5" side="left" x_offset="0" y_offset="${leg_radius}" yaw="${pi / 2}" colour="cyan"/>
+  <xacro:leg name="leg5" side="left" x_offset="0" y_offset="${middle_leg_y}" yaw="${pi / 2}" colour="cyan"/>
   <!-- Front left -->
-  <xacro:leg name="leg6" side="left" x_offset="${corner_offset}" y_offset="${corner_offset}" yaw="${pi / 4}" colour="magenta"/>
+  <xacro:leg name="leg6" side="left" x_offset="${corner_leg_x}" y_offset="${corner_leg_y}" yaw="${pi / 4}" colour="magenta"/>
   <!-- ================= SENSORS ================= -->
   <gazebo reference="camera_link">
